File: drive-download-20241228T173334Z-001/Final_project_rbree.kicad_pcb (KiCad board)
At the start: 2 copper layers, 48 parts, among them J1 Conn_01x02_Pin, J2 Conn_01x02_Pin, Q2 AO3401A, Q3 MMBT3904, U1 TL431, U2 LTV-817, U3 B1212, U4 2N7002, U7 NE555

Commit message: Add files via upload
Parts:
- moved R13 63.7 mm to (161.8, 93.3)
- moved U4 63.6 mm to (186.2, 75.5)
- moved U2 59.6 mm to (168.5, 93.9)
- moved Q2 55.8 mm to (199.1, 110.4)
- moved R19 52.3 mm to (186.1, 105.4)
- moved R14 50.4 mm to (181.2, 75.4), turned to -90 degrees
- moved R15 49.5 mm to (190.5, 92.4)
- moved Q3 49.4 mm to (185.6, 111.1)
- moved C4 46.4 mm to (146.0, 115.0)
- moved R21 44.2 mm to (193.0, 105.4), turned to 180 degrees
- moved R20 42.2 mm to (193.1, 100.4)
- moved H4 42.1 mm to (203.0, 139.0)
- moved R18 41.3 mm to (184.6, 89.0), turned to 90 degrees
- moved C1 40.4 mm to (140.2, 104.9)
- moved R1 40.4 mm to (127.2, 100.9)
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Routing:
- net VCC: track 13.1 -> 178.4 mm
- net GND: track 96.8 -> 214.8 mm
- net GLV-: track 39.8 -> 145.9 mm
- net +12V: track 10.2 -> 85.5 mm
- net /RED+: track 0.00 -> 32.0 mm
- net Net-(U4-G): track 0.00 -> 28.0 mm
- net Net-(Q3-B): track 0.00 -> 20.7 mm
- net Net-(U7-THR): track 0.00 -> 20.1 mm, vias 0 -> 2
- net Net-(U4-D): track 0.00 -> 19.6 mm
- net /Vref: track 23.1 -> 40.3 mm, vias 0 -> 2
- net Net-(LM1-Pad7): track 6.67 -> 18.0 mm
- net Net-(Q2-G): track 0.00 -> 10.6 mm
- net Net-(U7-DIS): track 0.00 -> 8.55 mm
- net Net-(Q3-C): track 0.00 -> 5.81 mm
- net Net-(D3-K): track 0.00 -> 5.05 mm
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- added copper zone on B.Cu, net GLV-
- added copper zone on F.Cu, net GLV-
Other:
- board outline added: 100 x 80 mm
